File: KiCad/RocketryFlightComputer_v0.1/RocketryFlightComputer_v0.1.kicad_sch (KiCad schematic)
At the start: 15 parts, among them J1 USB_C_Receptacle, Q1 BSS806NH6327XTSA1, Q2 BSS806NH6327XTSA1, Q3 BSS806NH6327XTSA1, U1 STM32U545RET6Q, U2 SX1262IMLTRT, U3 W25N01GWZEIG, U4 BME680, U5 MMC5633NJL, U6 TLV77118PDBVR, U7 ICM-20602, U8 TPS63070RNMR, U9 EVA-M8M-0, Y1 END4263D-32M, Y2 SIT1552AI-JE-DCC-32.768E

Commit message: finished power supply
Parts:
- added C1, C2: 10u, Capacitor_SMD:C_0805_2012Metric, symbol Device:C_Small
- added C3, C8: 10u, Capacitor_SMD:C_0603_1608Metric, symbol Device:C_Small
- added C4: 100n, Capacitor_SMD:C_0402_1005Metric, symbol Device:C_Small
- added C5, C6, C7: 22u, Capacitor_SMD:C_0805_2012Metric, symbol Device:C_Small
- added J2: Conn_Coaxial, Connector_Coaxial:U.FL_Hirose_U.FL-R-SMT-1_Vertical, symbol Connector:Conn_Coaxial
- added J3: DEPLOYMENT, TerminalBlock:TerminalBlock_Xinya_XY308-2.54-4P_1x04_P2.54mm_Horizontal, symbol Connector:Screw_Terminal_01x04
- added J4: POWER_IN, TerminalBlock:TerminalBlock_Xinya_XY308-2.54-2P_1x02_P2.54mm_Horizontal, symbol Connector:Screw_Terminal_01x02
- added L1: ETQ-P3M1R5KVP, Inductor_SMD:L_Vishay_IHLP-1212, symbol ETQ-P3M1R5KVP:ETQ-P3M1R5KVP
- added R1: 10k, Resistor_SMD:R_0402_1005Metric, symbol Device:R
- added R2: 470k, Resistor_SMD:R_0402_1005Metric, symbol Device:R_Small
- added R3: 150k, Resistor_SMD:R_0402_1005Metric, symbol Device:R_Small
- added R4: 100k, Resistor_SMD:R_0402_1005Metric, symbol Device:R_Small
- U9: footprint EVA-M8M-0:LGA43R65P9X9_700X700X116 -> LGA43R65P9X9_700X700X116
Connections:
- net VDD: now reaches U1.1 (VBAT)
- net VDD: now also U1.13 (VDDA), U1.19 (VDD), U1.29 (VDDSMPS), U1.31 (VDD11), U1.33 (VDD), U1.48 (VDDUSB), U1.62 (VDD11), U1.64 (VDD), U8.7 (VOUT), U8.8 (VOUT), C5.1, C6.1, C7.1, C8.1, R2.1, R4.1
- net GND: now reaches U1.12 (VSSA)
- net GND: now also U1.18 (VSS), U1.30 (VSSSMPS), U1.32 (VSS), U1.47 (VSS), U1.63 (VSS), U8.10 (PGND), U8.15 (VSEL), U8.4 (GND), U8.6 (FB2), C1.2, C2.2, C3.2, C4.1, C5.2, C6.2, C7.2, C8.2, J2.2 (Ext), J4.1 (Pin_1), R3.1
- net at U8.1 (PS_SYNC): now also U8.14 (EN), R1.2
- net at U8.11 (L1): now also L1.2
- net at U8.12 (VIN): now also U8.13 (VIN), C1.1, C2.1, C3.1, J4.2 (Pin_2), R1.1
- net at U8.2 (PG): now also R4.2
- net at U8.3 (VAUX): now also C4.2
- net at U8.5 (FB): now also R2.2, R3.2
- net at U8.9 (L2): now also L1.1
- net at U2.23 (RFO): now also J2.1 (In)

Commit message: Finished Board v0.1
Parts:
- removed J1: USB_C_Receptacle, Connector_USB:USB_C_Receptacle_Amphenol_12401548E4-2A, symbol Connector:USB_C_Receptacle
- removed Y1: END4263D-32M, Oscillator:Oscillator_DIP-14, symbol Oscillator:TCXO-14
- removed Y2: SIT1552AI-JE-DCC-32.768E, Oscillator:Oscillator_DIP-14, symbol Oscillator:TCXO-14
- added C10, C9: 2.2u, Resistor_SMD:R_0402_1005Metric, symbol Device:C_Small
- added C11: 10p, Resistor_SMD:R_0402_1005Metric, symbol Device:C_Small
- added C12: 100n, Resistor_SMD:R_0402_1005Metric, symbol Device:C_Small
- added C13: 470u, Capacitor_SMD:C_0402_1005Metric, symbol Device:C_Small
- added C14, C15, C16, C17: 0, Capacitor_SMD:C_0402_1005Metric, symbol Device:C_Small
- added C18: 1.5p, Capacitor_SMD:C_0201_0603Metric, symbol Device:C_Small
- added C19, C20: 1p, Capacitor_SMD:C_0201_0603Metric, symbol Device:C_Small
- added C21: 100p, Capacitor_SMD:C_0201_0603Metric, symbol Device:C_Small
- added C22, C27, C28, C29, C30: 100n, Capacitor_SMD:C_0201_0603Metric, symbol Device:C_Small
- added C23, C24, C33, C34, C35: 10u, Capacitor_SMD:C_0201_0603Metric, symbol Device:C_Small
- added C25: 4.7u, Capacitor_SMD:C_0201_0603Metric, symbol Device:C_Small
- added C26, C31: 1u, Capacitor_SMD:C_0201_0603Metric, symbol Device:C_Small
- added C32, C36, C37: 2.2u, Capacitor_SMD:C_0201_0603Metric, symbol Device:C_Small
- added D1: LED, LED_SMD:LED_0402_1005Metric, symbol Device:LED
- added J1: Conn_01x06_Pin, Connector_PinHeader_1.00mm:PinHeader_1x06_P1.00mm_Vertical_SMD_Pin1Left, symbol Connector:Conn_01x06_Pin
- added J5: USB_C_Receptacle_USB2.0_16P, Connector_USB:USB_C_Receptacle_GCT_USB4105-xx-A_16P_TopMnt_Horizontal, symbol Connector:USB_C_Receptacle_USB2.0_16P
- added J6: Conn_Coaxial, Connector_Coaxial:U.FL_Hirose_U.FL-R-SMT-1_Vertical, symbol Connector:Conn_Coaxial
- added L2: 2.2u, Capacitor_SMD:C_0805_2012Metric, symbol Device:L
- added L3: 3.9n, Inductor_SMD:L_0201_0603Metric, symbol Device:L
- added L4: 6.8n, Inductor_SMD:L_0201_0603Metric, symbol Device:L
- added L5: 8.2n, Inductor_SMD:L_0201_0603Metric, symbol Device:L
- added Q4: BSS806NH6327XTSA1, Package_TO_SOT_SMD:SOT-23, symbol Transistor_FET:BSS123
- added R10, R11, R12: 10k, Resistor_SMD:R_0402_1005Metric, symbol Device:R_Small
- added R13: 220, Resistor_SMD:R_0402_1005Metric, symbol Device:R_Small
- added R14, R15: 10k, Capacitor_SMD:C_0402_1005Metric, symbol Device:R
- added R16, R17: 0, Resistor_SMD:R_0402_1005Metric, symbol Device:R_Small
- added R18: 10k, Resistor_SMD:R_0201_0603Metric, symbol Device:R
- added R19: 100k, Resistor_SMD:R_0201_0603Metric, symbol Device:R_Small
- added R20: 330, Resistor_SMD:R_0201_0603Metric, symbol Device:R_Small
- added R5, R6: 5.1k, Resistor_SMD:R_0402_1005Metric, symbol Device:R_Small
- added R7, R8, R9: 100, Resistor_SMD:R_0402_1005Metric, symbol Device:R
- added S1, S2: TS21-34-035-BK-160-SMT-TR, Footprints:SW_TS21-34-035-BK-160-SMT-TR, symbol TS21-34-035-BK-160-SMT-TR:TS21-34-035-BK-160-SMT-TR
- added U10: SKY13453-385LF, QFN_453-385LF_SKY, symbol SKY13453-385LF:SKY13453-385LF
- added U11: TLV75733PDBV, Package_TO_SOT_SMD:SOT-23-5, symbol Regulator_Linear:TLV75733PDBV
- added XTAL1: SIT1552AI-JE-DCC-32.768E, BGA4_SiT1532_SIT, symbol 2026-05-09_18-51-59:SIT1552AI-JE-DCC-32.768E
- added Y1: ECS-2520MV-xxx-xx, Crystal:Crystal_SMD_SeikoEpson_FA128-4Pin_2.0x1.6mm, symbol Oscillator:ECS-2520MV-xxx-xx
- added Y2: TG2520SMN, Oscillator:Oscillator_SMD_SeikoEpson_TG2520SMN-xxx-xxxxxx-4Pin_2.5x2.0mm, symbol Oscillator:TG2520SMN-xx.xxxxxxMhz-xxxxNM
- J3: footprint TerminalBlock:TerminalBlock_Xinya_XY308-2.54-4P_1x04_P2.54mm_Horizontal -> TerminalBlock_Phoenix:TerminalBlock_Phoenix_MPT-0,5-4-2.54_1x04_P2.54mm_Horizontal
- J4: footprint TerminalBlock:TerminalBlock_Xinya_XY308-2.54-2P_1x02_P2.54mm_Horizontal -> TerminalBlock_Phoenix:TerminalBlock_Phoenix_MPT-0,5-2-2.54_1x02_P2.54mm_Horizontal
- U8: footprint RNM0015A -> Footprints:RNM0015A
- U9: footprint LGA43R65P9X9_700X700X116 -> Footprints:LGA43R65P9X9_700X700X116
Connections:
- net GND: now also Q1.2 (S), Q2.2 (S), Q3.2 (S), U2.2 (GND), U2.20 (GND), U2.25 (GND), U2.5 (GND), U2.8 (GND), U3.4 (GND), U3.9 (EP), U4.1 (GND), U4.7 (GND), U5.A1 (VSA), U6.2 (GND), U6.4 (GND), U7.10 (GND), U7.11 (GND), U7.12 (GND), U7.13 (GND), U7.15 (GND), U7.9 (GND), U9.18 (GND__1), U9.2 (GND), U9.32 (D_SEL), U9.37 (GND__2), U9.38 (GND__3), U9.39 (GND__4), U9.40 (GND__5), U9.41 (GND__6), U9.42 (GND__7), U9.43 (GND__8), U9.7 (VDD_USB), U9.9 (RTC_I), C10.2, C12.2, C13.2, C14.2, C15.2, C16.2, C17.2, C18.2, C19.2, C21.2, C22.2, C23.2, C24.2, C25.2, C26.2, C27.2, C28.2, C29.2, C30.2, C31.2, C32.2, C33.2, C34.2, C35.2, C36.2, C37.2, C9.2, D1.1 (K), J1.3 (Pin_3), J5.A1 (GND), J5.A12 (GND), J5.B1 (GND), J5.B12 (GND), J5.S1 (SHIELD), J6.2 (Ext), L5.2, Q4.2 (S), R10.2, R11.2, R12.2, R15.2, R5.1, R6.2, S2.1, S2.2, U10.3 (GND), U11.2 (GND), XTAL1.1 (GND), XTAL1.4 (GND), Y1.2 (GND), Y2.2 (GND)
- net VDD: now also U2.1 (VDD_IN), U2.10 (VBAT), U2.11 (VBAT_IO), U3.8 (VCC), U4.6 (VDDIO), U4.8 (VDD), U5.B1 (VDD), U6.1 (IN), U6.3 (EN), U7.1 (VDDIO), U7.16 (VDD), U9.20 (VCC_IO), C22.1, C23.1, C24.1, C25.1, C26.1, C27.1, C28.1, C29.1, C30.1, C31.1, C32.1, C33.1, C34.1, C37.1, J1.1 (Pin_1), R14.1, R20.1, S1.1, S1.2, U10.1 (VDD), U11.5 (OUT), XTAL1.3 (VDD), Y1.4 (VDD); no longer U1.31 (VDD11), U1.62 (VDD11)
- net +BATT: now reaches J3.1 (Pin_1)
- net +BATT: now also C1.1, C2.1, C3.1, J4.2 (Pin_2), R1.1, U8.12 (VIN), U8.13 (VIN), R19.1
- net at J3.2 (Pin_2): now also Q1.3 (D)
- net at J3.3 (Pin_3): now also Q2.3 (D)
- net at J3.4 (Pin_4): now also Q3.3 (D)
- net +1V8: now reaches U6.5 (OUT)
- net +1V8: now also U9.19 (VCC), C35.1
- net SCL: now reaches U5.A2 (SCL)
- net SCL: now also U1.8 (PC0)
- net SDA: now reaches U5.B2 (SDA)
- net SDA: now also U1.9 (PC1)
- net at J2.1 (In): now also C14.1, R16.2; no longer U2.23 (RFO)
- net QSPI_CSN: now reaches U1.16 (PA2)
- net QSPI_CSN: now also U3.1 (~{CS})
- net QSPI_CLK: now reaches U1.17 (PA3)
- net QSPI_CLK: now also U3.6 (CLK)
- net QSPI_D3: now reaches U1.22 (PA6)
- net QSPI_D3: now also U3.7 (~{HOLD}/~{RESET}/IO_{3})
- net QSPI_D2: now reaches U1.23 (PA7)
- net QSPI_D2: now also U3.3 (~{WP}/IO_{2})
- net QSPI_D1: now reaches U1.24 (PB0)
- net QSPI_D1: now also U3.2 (DO/IO_{1})
- net QSPI_D0: now reaches U1.25 (PB1)
- net QSPI_D0: now also U3.5 (DI/IO_{0})
- net SX_NRST: now reaches U1.26 (PB2)
- net SX_NRST: now also U2.15 (~{RESET})
- net SX_BUSY: now reaches U1.27 (PB10)
- net SX_BUSY: now also U2.14 (BUSY)
- net V_SMPS: now reaches U1.28 (VLXSMPS)
- net V_SMPS: now also L2.1
- net at U1.3 (PC14): now also XTAL1.2 (CLK_OUT)
- net SCK: now reaches U1.34 (PB13)
- net SCK: now also U2.18 (SCK), U4.4 (SCK), U7.2 (SCL/SPC), U9.29 (SCL/SPI_CLK)
- net MISO: now reaches U1.35 (PB14)
- net MISO: now also U2.16 (MISO), U4.5 (SDO), U7.4 (SAO/SD0), U9.16 (TXD/SPI_MISO)
- net MOSI: now reaches U1.36 (PB15)
- net MOSI: now also U2.17 (MOSI), U4.3 (SDI), U7.3 (SDA/SDI), U9.15 (RXD/SPI_MOSI)
- net SX_CSN: now reaches U1.37 (PC6)
- net SX_CSN: now also U2.19 (NSS)
- net USB_D-: now reaches U1.44 (PA11)
- net USB_D-: now also J5.A7 (D-), J5.B7 (D-)
- net USB_D+: now reaches U1.45 (PA12)
- net USB_D+: now also J5.A6 (D+), J5.B6 (D+)
- net SWDIO: now reaches U1.46 (PA13)
- net SWDIO: now also J1.4 (Pin_4)
- net SWCLK: now reaches U1.49 (PA14)
- net SWCLK: now also J1.2 (Pin_2)
- net at U1.5 (PH0): now also Y1.3 (OUT)
- net SWO: now reaches U1.55 (PB3)
- net SWO: now also J1.6 (Pin_6)
- net BOOT0: now reaches U1.60 (PH3)
- net BOOT0: now also R15.1, S1.3, S1.4
- net NRST: now reaches U1.7 (NRST)
- net NRST: now also J1.5 (Pin_5), R14.2, S2.3, S2.4
- net ICM_CSN: now reaches U7.5 (~{CS})
- net at Q1.1 (G): now also R10.1, R7.2
- net BME_CSN: now reaches U4.2 (CSB)
- net at R1.2, U8.1 (PS_SYNC): no longer U8.14 (EN)
- net at Q3.1 (G): now also R12.1, R9.2
- net at U9.1 (RF_IN): now also C17.1, R17.1
- net GPS_CSN: now reaches U9.30 (SDA/SPI_CS_N)
- net at Q2.1 (G): now also R11.1, R8.2
- net RF_SW_CTRL: now reaches U2.12 (DIO2)
- net RF_SW_CTRL: now also U10.5 (VCTL)
- net SX_IRQ: now reaches U2.13 (DIO1)
- net RFI_P: now reaches U2.21 (RFI_P)
- net RFI_P: now also C20.2, L5.1
- net RFI_N: now reaches U2.22 (RFI_N)
- net RFI_N: now also C21.1
- net VR_PA: now reaches U2.24 (VR_PA)
- net at U2.3 (XTA): now also C11.2
- net at U2.6 (DIO3): now also C12.1, Y2.4 (Vcc)
- net at U2.7 (VREG): now also C13.1
- new net: J5.A5 (CC1), R5.2
- new net: C18.1, L3.2, L4.1
- new net: C19.1, L4.2, U10.2 (RF1)
- new net: C10.1, C9.1, L2.2, U1.31 (VDD11), U1.62 (VDD11)
- new net: C15.1, R16.1, U10.6 (RFC)
- new net: J5.B5 (CC2), R6.1
- new net: C16.1, J6.1 (In), R17.2
- new net: R13.2, Y2.3 (OUT)
- new net: C20.1, U10.4 (RF2)
- new net: D1.2 (A), R20.2
- new net: C11.1, R13.1
- new net: Q4.1 (G), R18.2
- new net 3V3_EN: Q4.3 (D), R19.2, U8.14 (EN)
- new net DEPLOY1: R7.1
- new net DEPLOY2: R8.1
- new net DEPLOY3: R9.1
- new net RF_O: L3.1, U2.23 (RFO)
- new net USB_VBUS: C36.1, J5.A4 (VBUS), J5.A9 (VBUS), J5.B4 (VBUS), J5.B9 (VBUS), R18.1, U11.1 (IN), U11.3 (EN)
- no-connect marks 0 -> 24
Other:
- moved on the sheet: J3, Q1, Q2, Q3, U5, U9
